Commit message: feature(simulation): Manual controlled drone and new assets
==============================================================
Description:
==============================================================
 It adds a manual controller to the drone and new assets for the simulation.
 New 3D models are added for the drone.
 The drone can now be controlled manually using the keyboard.

	new file:   ../PyBullet_Quickstart_Guide.pdf
        - Added a quick start guide for PyBullet

	new file:   ../assets/cf2_modern.dae
        - Added a new 3D model for the drone
        - The new model is more modern and has a better look
        - no changes in the dynamics of the drone

	modified:   ../assets/cf2x.urdf
        - Updated the URDF file to use the new 3D model

	new file:   ../assets/save/cf2.dae
    new file:   ../assets/save/cf2p.urdf
	new file:   ../assets/save/cf2x.urdf
        - backup of the old 3D model

	new file:   cf2_color.dae
        - Experimental 3D model with color

	modified:   simulation.py
        -  Added manual controller for the drone
        -  The drone can now be controlled using the keyboard
        -  The manual controller allows for more precise control of the drone
        -  The manual controller can be used for testing and debugging purposes
        - Added new function for image capture
        - this function captures the image from the drone's camera and uses
            it in a separate window (still very slow)
        - Fixed trajectory for the automous drones that where stopped

File: gym_pybullet_drones/assets/cf2x.urdf (robot description, URDF)
Before this commit: robot cf2, 6 links, 5 joints
Links:
- link base_link: geometry collision cylinder length=.025 radius=.06; visual mesh filename=./cf2_modern.dae scale=1 1 1

File: gym_pybullet_drones/search_rescue/cf2x.urdf (robot description, URDF)
Before this commit: robot cf2, 6 links, 5 joints
Links:
- link base_link: geometry collision cylinder length=.025 radius=.06; visual mesh filename=./cf2_new.dae scale=1 1 1

Commit message: New functions to the model included classes but still not fully implemented manual controler working
==============================================================
Description:
==============================================================

File: gym_pybullet_drones/assets/cf2x.urdf (robot description, URDF)
Before this commit: robot cf2, 6 links, 5 joints
Links:
- link base_link: geometry collision cylinder length=.025 radius=.06; visual mesh filename=./cf2.dae scale=1 1 1

File: gym_pybullet_drones/search_rescue/cf2x.urdf (robot description, URDF)
Before this commit: robot cf2, 6 links, 5 joints
Links:
- link base_link: geometry collision cylinder length=.025 radius=.06; visual mesh filename=./cf2.dae scale=1 1 1
